File: balanced-modulator.kicad_pcb (KiCad board)
At the start: 2 copper layers, 11 parts, among them J1 Conn_02x05_Odd_Even

Commit message: board + readme
Parts:
- added C3: 100n, Capacitor_SMD:C_0805_2012Metric, F.Cu at (145.1, 83.9)
- added C4: 100u 16V, Capacitor_THT:CP_Radial_D5.0mm_P2.50mm, B.Cu at (125.1, 91.0)
- added C5: 1u box, Eurorack:C_Rect_Horizontal_L7.2mm_W11, B.Cu at (122.7, 115.2)
- added C6: 1u box, Eurorack:C_Rect_Horizontal_L7.2mm_W11, B.Cu at (110.0, 115.2)
- added C7: 1u box, Eurorack:C_Rect_Horizontal_L7.2mm_W11, B.Cu at (135.4, 115.2)
- added H10: MountingHole, MountingHole:MountingHole_2.7mm_M2.5, F.Cu at (149.4, 108.3)
- added H11: MountingHole, MountingHole:MountingHole_2.7mm_M2.5, F.Cu at (149.4, 83.2)
- added H5: carrier, Eurorack:Mech-AudioJack-Hole-Input, F.Cu at (102.7, 146.7)
- added H6: modulating, Eurorack:Mech-AudioJack-Hole-Input, F.Cu at (102.7, 135.5)
- added H7: out, Eurorack:Mech-AudioJack-Hole-Output, F.Cu at (141.2, 137.9)
- added H8: MountingHole, MountingHole:MountingHole_2.7mm_M2.5, F.Cu at (94.7, 107.3)
- added H9: MountingHole, MountingHole:MountingHole_2.7mm_M2.5, F.Cu at (94.7, 82.2)
- added J10: out, Eurorack:AudioJack2_Tayda_A-2566, F.Cu at (141.2, 104.3)
- added J2: Conn_01x03_Socket, Connector_PinSocket_2.54mm:PinSocket_1x03_P2.54mm_Vertical, F.Cu at (150.0, 73.3)
- added J3: Conn_01x03_Pin, Connector_PinHeader_2.54mm:PinHeader_1x03_P2.54mm_Vertical, B.Cu at (150.0, 98.3)
- added J4: Conn_01x03_Pin, Connector_PinHeader_2.54mm:PinHeader_1x03_P2.54mm_Vertical, B.Cu at (94.1, 112.1)
- added J5: Conn_01x03_Socket, Connector_PinSocket_2.54mm:PinSocket_1x03_P2.54mm_Vertical, F.Cu at (94.1, 87.1)
- added J8: carrier, Eurorack:AudioJack2_Tayda_A-2566, F.Cu at (102.7, 101.9)
- added J9: modulating, Eurorack:AudioJack2_Tayda_A-2566, F.Cu at (102.7, 113.1)
- added JP1: Jumper_3_Bridged12, Connector_PinHeader_2.54mm:PinHeader_1x03_P2.54mm_Horizontal, B.Cu at (124.6, 109.6)
- added JP2: Jumper_3_Bridged12, Connector_PinHeader_2.54mm:PinHeader_1x03_P2.54mm_Horizontal, B.Cu at (116.0, 109.6)
- added JP3: Jumper_3_Bridged12, Connector_PinHeader_2.54mm:PinHeader_1x03_P2.54mm_Horizontal, B.Cu at (133.3, 109.6)
- added R10: 180K, Resistor_SMD:R_0805_2012Metric, F.Cu at (119.7, 76.6)
- added R11: 2.7K, Resistor_SMD:R_0805_2012Metric, F.Cu at (117.5, 76.6)
- added R12: 6.8K, Resistor_SMD:R_0805_2012Metric, F.Cu at (122.0, 76.6)
- added R13: 6.8K, Resistor_SMD:R_0805_2012Metric, F.Cu at (123.5, 84.8)
- added R14: 2.7K, Resistor_SMD:R_0805_2012Metric, F.Cu at (123.5, 81.0)
- added R15: 6.8K, Resistor_SMD:R_0805_2012Metric, F.Cu at (115.2, 76.6)
- added R16: 15K, Resistor_SMD:R_0805_2012Metric, F.Cu at (141.6, 76.9)
- added R17: 15K, Resistor_SMD:R_0805_2012Metric, F.Cu at (139.3, 76.9)
- added R18: 1.2K, Resistor_SMD:R_0805_2012Metric, F.Cu at (112.9, 76.6)
- added R19: 1.2K, Resistor_SMD:R_0805_2012Metric, F.Cu at (136.5, 81.4)
- added R20: 15K, Resistor_SMD:R_0805_2012Metric, F.Cu at (137.0, 76.9)
- added R21: 15K, Resistor_SMD:R_0805_2012Metric, F.Cu at (143.9, 76.9)
- added R22: 10K, Resistor_SMD:R_0805_2012Metric, F.Cu at (140.8, 89.1)
- added R23: 68K, Resistor_SMD:R_0805_2012Metric, F.Cu at (138.5, 89.1)
- added R24: 1K, Resistor_SMD:R_0805_2012Metric, F.Cu at (143.1, 89.1)
- added R3: 180K, Resistor_SMD:R_0805_2012Metric, F.Cu at (112.9, 88.8)
- added R4: 12K, Resistor_SMD:R_0805_2012Metric, F.Cu at (115.2, 88.8)
- added R5: 2.7K, Resistor_SMD:R_0805_2012Metric, F.Cu at (117.5, 88.8)
- added R6: 2.7K, Resistor_SMD:R_0805_2012Metric, F.Cu at (119.7, 88.8)
- added R7: 12K, Resistor_SMD:R_0805_2012Metric, F.Cu at (122.0, 88.8)
- added R8: 1.5K, Resistor_SMD:R_0805_2012Metric, F.Cu at (127.1, 81.0)
- added R9: 1.5K, Resistor_SMD:R_0805_2012Metric, F.Cu at (127.1, 84.8)
- added RV1: 500, Potentiometer_THT:Potentiometer_Bourns_3296W_Vertical, B.Cu at (132.2, 86.1)
- added RV2: 200, Potentiometer_THT:Potentiometer_Bourns_3296W_Vertical, B.Cu at (132.2, 75.4)
- added U1: MC1496, Package_SO:SOIC-14_3.9x8.7mm_P1.27mm, F.Cu at (116.7, 82.7)
- added U2: TL072, Package_SO:SOIC-8_3.9x4.9mm_P1.27mm, F.Cu at (140.9, 82.9)
- D1, D2, R1, R2: moved to F.Cu
- moved H3 172.2 mm to (147.4, 158.2)
- moved H2 151.0 mm to (147.4, 124.6)
- moved H4 141.0 mm to (96.8, 158.2)
- moved H1 123.1 mm to (96.8, 124.6)
- moved R1 38.4 mm to (107.0, 84.0)
- moved R2 38.4 mm to (107.0, 81.5)
- moved D2 38.0 mm to (107.2, 87.8)
- moved D1 37.9 mm to (107.1, 77.7)
- moved J1 36.9 mm to (103.6, 77.7)
- moved C1 36.8 mm to (110.0, 89.3), turned to 90 degrees
- moved C2 22.5 mm to (110.0, 78.6)
Routing:
- net GND: track 0.00 -> 60.0 mm, vias 0 -> 7
- net -12V: track 15.8 -> 75.1 mm, vias 0 -> 1
- net +12V: track 14.0 -> 73.1 mm
- net /_B: track 0.00 -> 45.1 mm
- net Net-(R17-Pad1): track 0.00 -> 34.9 mm
- net Net-(R16-Pad2): track 0.00 -> 34.4 mm
- net /_A': track 0.00 -> 30.8 mm
- net /OUT_dc': track 0.00 -> 23.9 mm
- net /_B': track 0.00 -> 23.5 mm
- net /_OUT': track 0.00 -> 22.9 mm
- net /A_dc': track 0.00 -> 22.4 mm
- net Net-(R21-Pad2): track 0.00 -> 20.9 mm
- net Net-(R4-Pad2): track 0.00 -> 20.6 mm, vias 0 -> 1
- net /_A: track 0.00 -> 19.4 mm
- net /B_dc': track 0.00 -> 18.0 mm
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- added copper zone on B.Cu, net /FACE
- added copper zone on F.Cu, net /FACE
- added copper zone on B.Cu, net /GND'
- added copper zone on F.Cu, net /GND'
- added copper zone on B.Cu, net GND
- added copper zone on F.Cu, net GND
Other:
- board outline added: 60.6 x 89.7 mm
- board text added: "ac"
- board text added: "balanced modulator"
- board text added: "car"
- board text added: "carrier"
- board text added: "dc"
- board text added: "mod"
- board text added: "modulating"
- board text added: "out"
- board text added: "thismatters/balanced-modulator/v0"
- board text removed: "POWER"

Commit message: ready for v0 manu
Changed lines of the file:
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@@
   )
   (gr_text "thismatters/balanced-modulator/v0" (at 137.033 72.2122) (layer "B.SilkS")
-    (effects (font (size 1 1) (thickness 0.1)) (justify left mirror))
+    (effects (font (size 1 1) (thickness 0.15)) (justify left mirror))
   )
   (gr_text "balanced modulator" (at 122.809 160.401) (layer "F.SilkS")
@@
   )
   (gr_text "thismatters/balanced-modulator/v0" (at 109.7788 97.3074) (layer "F.SilkS")
-    (effects (font (size 1 1) (thickness 0.1)) (justify left))
+    (effects (font (size 1 1) (thickness 0.15)) (justify left))
   )
   (gr_text "carrier" (at 108.077 135.509) (layer "F.SilkS")
     (effects (font (size 2 1.75) (thickness 0.2) bold) (justify left))
   )
-  (gr_text "thismatters/balanced-modulator/v0" (at 92.71 127.254 -90) (layer "F.SilkS")
-    (effects (font (size 1 1) (thickness 0.1)) (justify left))
+  (gr_text "thismatters/balanced-modulator/v0" (at 92.71 127.254 270) (layer "F.SilkS")
+    (effects (font (size 1 1) (thickness 0.15)) (justify left))
   )
   (gr_text "modulating" (at 108.077 146.685) (layer "F.SilkS")
